File: Controlador_BLDC.kicad_sch (KiCad schematic)
At the start: 126 parts, among them IC1 AP1509-50SG-13, J1 Conn_01x03, J10 Conn_01x04_Pin, J11 Conn_01x02_Pin, J12 Conn_01x02_Pin, J13 Conn_01x02_Pin, J2 Conn_01x04_Pin, J3 Conn_01x04_Pin, J4 Conn_01x04_Pin, J5 Conn_01x04_Pin, J6 Conn_01x04_Pin, J7 Conn_01x07_Pin, J8 Conn_01x02_Pin, J9 Conn_01x02_Pin, U1 LM324, U2 LM324, U3 LMS8117AMP-3.3/NOPB, U4 LM339DR, U5 EK-TM4C123GXL, U6 IR2301SPBF, U7 IR2301SPBF, U8 IR2301SPBF

Commit message: Add files via upload
Parts:
- added CAHF1, CBHF1, CCHF1: 100nF 50V X7R, ESC_BLDC:C_1206_3216Metric_Pad1.33x1.80mm_HandSolder, symbol Device:C
- added C_U1, C_U2, C_U4: 100nF, ESC_BLDC:C_1206_3216Metric_Pad1.33x1.80mm_HandSolder, symbol Device:C
- added J_SPI: SPI_LSE2, ESC_BLDC:PinHeader_1x05_P2.54mm_Vertical, symbol Connector:Conn_01x05_Pin
- added TP_GND1, TP_GND2, TP_GND3: TP_GND, ESC_BLDC:PinHeader_1x01_P2.54mm_Vertical, symbol Connector:Conn_01x01_Pin
- added unit 4 of U2
- added unit 3 of U2
- CADES1, CBDES1, CCDES1: value ~ -> 10uF 25V X5R; footprint Capacitor_SMD:C_1206_3216Metric_Pad1.33x1.80mm_HandSolder -> ESC_BLDC:C_1206_3216Metric_Pad1.33x1.80mm_HandSolder
- CADES2, CBDES2, CCDES2: value ~ -> 47uF 25V; footprint Capacitor_SMD:C_Elec_6.3x5.8 -> ESC_BLDC:CP_Elec_6.3x7.7; symbol Device:C -> Device:C_Polarized
- CAH1, CAL1, CBH1, CBL1, CCH1, CCL1, CbypassA1, CbypassB1, CbypassC1: value ~ -> 100pF C0G; footprint Capacitor_SMD:C_1206_3216Metric_Pad1.33x1.80mm_HandSolder -> ESC_BLDC:C_1206_3216Metric_Pad1.33x1.80mm_HandSolder
- CA_BOOT1, CB_BOOT1, CC_BOOT1: value ~ -> 1uF 50V X7R; footprint Capacitor_SMD:C_Elec_6.3x5.8 -> ESC_BLDC:C_1206_3216Metric_Pad1.33x1.80mm_HandSolder
- CBEM_A1, CBEM_B1, CBEM_C1, CDiv1: value ~ -> 22nF 5%; footprint Capacitor_SMD:C_1206_3216Metric_Pad1.33x1.80mm_HandSolder -> ESC_BLDC:C_1206_3216Metric_Pad1.33x1.80mm_HandSolder
- CDES1: value 100nF -> 470uF 25V; footprint Capacitor_THT:C_Radial_D12.5mm_H20.0mm_P5.00mm -> ESC_BLDC:CP_Radial_D10.0mm_P5.00mm; symbol Device:C -> Device:C_Polarized
- CDES2: value ~ -> 10uF 10V X5R; footprint Capacitor_SMD:C_1206_3216Metric_Pad1.33x1.80mm_HandSolder -> ESC_BLDC:C_1206_3216Metric_Pad1.33x1.80mm_HandSolder
- CDESPOT1, CPOT3: footprint Capacitor_SMD:C_1206_3216Metric_Pad1.33x1.80mm_HandSolder -> ESC_BLDC:C_1206_3216Metric_Pad1.33x1.80mm_HandSolder
- CPOT1: value 10uF -> 10uF 25V X5R; footprint Capacitor_SMD:C_1206_3216Metric_Pad1.33x1.80mm_HandSolder -> ESC_BLDC:C_1206_3216Metric_Pad1.33x1.80mm_HandSolder
- CPOT2: value 10uF -> 220uF 10V; footprint Capacitor_SMD:C_1206_3216Metric_Pad1.33x1.80mm_HandSolder -> ESC_BLDC:CP_Elec_6.3x7.7; symbol Device:C -> Device:C_Polarized
- CPOT4: value 10uF -> 10uF 16V X5R; footprint Capacitor_SMD:C_1206_3216Metric_Pad1.33x1.80mm_HandSolder -> ESC_BLDC:C_1206_3216Metric_Pad1.33x1.80mm_HandSolder
- CPOT5: value 10uF -> 10uF 10V tantal (ESR 0.5-5R); footprint Capacitor_SMD:C_1206_3216Metric_Pad1.33x1.80mm_HandSolder -> ESC_BLDC:CP_EIA-3216-18_Kemet-A_Pad1.58x1.35mm_HandSolder; symbol Device:C -> Device:C_Polarized
- D1: footprint Diode_THT:D_DO-41_SOD81_P10.16mm_Horizontal -> ESC_BLDC:D_DO-41_SOD81_P10.16mm_Horizontal
- D2, D3, D4: footprint Diode_THT:D_DO-35_SOD27_P7.62mm_Horizontal -> ESC_BLDC:D_DO-35_SOD27_P7.62mm_Horizontal
- IC1: footprint AP1509-50SG-13:SOIC127P600X170-8N -> ESC_BLDC:SOIC-8_3.9x4.9mm_P1.27mm
- J1: value Conn_01x03 -> MOTOR; footprint (none) -> ESC_BLDC:TerminalBlock_Phoenix_MKDS-1,5-3-5.08_1x03_P5.08mm_Horizontal
- J10: value Conn_01x04_Pin -> TP_BUCK; footprint (none) -> ESC_BLDC:PinHeader_1x04_P2.54mm_Vertical
- J11: value Conn_01x02_Pin -> TP_+3V3; footprint (none) -> ESC_BLDC:PinHeader_1x02_P2.54mm_Vertical
- J12: value Conn_01x02_Pin -> TP_+5V; footprint (none) -> ESC_BLDC:PinHeader_1x02_P2.54mm_Vertical
- J13: value Conn_01x02_Pin -> TP_VCC; footprint (none) -> ESC_BLDC:PinHeader_1x02_P2.54mm_Vertical
- J2: value Conn_01x04_Pin -> TP_SENSOR; footprint (none) -> ESC_BLDC:PinHeader_1x04_P2.54mm_Vertical
- J3: value Conn_01x04_Pin -> TP_BEMF; footprint (none) -> ESC_BLDC:PinHeader_1x04_P2.54mm_Vertical
- J4: value Conn_01x04_Pin -> TP_VREF_ADC; footprint (none) -> ESC_BLDC:PinHeader_1x04_P2.54mm_Vertical
- J5: value Conn_01x04_Pin -> TP_VNDIV; footprint (none) -> ESC_BLDC:PinHeader_1x04_P2.54mm_Vertical
- J6: value Conn_01x04_Pin -> TP_BEMFD; footprint (none) -> ESC_BLDC:PinHeader_1x04_P2.54mm_Vertical
- J7: value Conn_01x07_Pin -> TP_OPAMP; footprint (none) -> ESC_BLDC:PinHeader_1x07_P2.54mm_Vertical
- J8: value Conn_01x02_Pin -> TP_NEUTRE; footprint (none) -> ESC_BLDC:PinHeader_1x02_P2.54mm_Vertical
- J9: value Conn_01x02_Pin -> TP_DUTY; footprint (none) -> ESC_BLDC:PinHeader_1x02_P2.54mm_Vertical
- J_DC1: value ~ -> 12V_IN; footprint TerminalBlock_Phoenix:TerminalBlock_Phoenix_MKDS-1,5-2-5.08_1x02_P5.08mm_Horizontal -> ESC_BLDC:TerminalBlock_Phoenix_MKDS-1,5-2-5.08_1x02_P5.08mm_Horizontal
- J_TPA1: value PART_A -> TP_FASE_A; footprint Connector_PinHeader_2.54mm:PinHeader_1x05_P2.54mm_Vertical -> ESC_BLDC:PinHeader_1x05_P2.54mm_Vertical
- J_TPA2: value PART_A -> TP_FASE_B; footprint Connector_PinHeader_2.54mm:PinHeader_1x05_P2.54mm_Vertical -> ESC_BLDC:PinHeader_1x05_P2.54mm_Vertical
- J_TPA3: value PART_A -> TP_FASE_C; footprint Connector_PinHeader_2.54mm:PinHeader_1x05_P2.54mm_Vertical -> ESC_BLDC:PinHeader_1x05_P2.54mm_Vertical
- J_VBA1: value V_BootDriverA -> TP_VBA; footprint Connector_PinHeader_2.54mm:PinHeader_1x01_P2.54mm_Vertical -> ESC_BLDC:PinHeader_1x01_P2.54mm_Vertical
- J_VBA2: value V_BootDriverA -> TP_VBB; footprint Connector_PinHeader_2.54mm:PinHeader_1x01_P2.54mm_Vertical -> ESC_BLDC:PinHeader_1x01_P2.54mm_Vertical
- J_VBA3: value V_BootDriverA -> TP_VBC; footprint Connector_PinHeader_2.54mm:PinHeader_1x01_P2.54mm_Vertical -> ESC_BLDC:PinHeader_1x01_P2.54mm_Vertical
- J_VBA4: value V_BootDriverA -> TP_FASE_A; footprint Connector_PinHeader_2.54mm:PinHeader_1x01_P2.54mm_Vertical -> ESC_BLDC:PinHeader_1x01_P2.54mm_Vertical
- J_VBA5: value V_BootDriverA -> TP_FASE_B; footprint Connector_PinHeader_2.54mm:PinHeader_1x01_P2.54mm_Vertical -> ESC_BLDC:PinHeader_1x01_P2.54mm_Vertical
- J_VBA6: value V_BootDriverA -> TP_FASE_C; footprint Connector_PinHeader_2.54mm:PinHeader_1x01_P2.54mm_Vertical -> ESC_BLDC:PinHeader_1x01_P2.54mm_Vertical
- L1: value SRN4018-4R7M -> 39uH SRN6045TA-390M; footprint SRN4018-4R7M:IND_BOURNS_SRN4018 -> ESC_BLDC:L_Bourns_SRN6045TA
- LED1: value LTL-4221N -> LTL-4221N (vermell); footprint LIB_LTL-4221N:LTL4221N -> ESC_BLDC:LED_D3.0mm
- MOSFET1, MOSFET2, MOSFET3, MOSFET4, MOSFET5, MOSFET6: footprint IRFR1205TRPBF:D-PAK_TO-252AA_INF -> ESC_BLDC:TO-252-2
- R1: footprint Resistor_SMD:R_1206_3216Metric_Pad1.30x1.75mm_HandSolder -> ESC_BLDC:R_1206_3216Metric_Pad1.30x1.75mm_HandSolder
- RAH1, RAL1, RBH1, RBL1, RCH1, RCL1, RGAH1, RGAL1, RGBH1, RGBL1, RGCH1, RGCL1: value ~ -> 33; footprint Resistor_SMD:R_1206_3216Metric_Pad1.30x1.75mm_HandSolder -> ESC_BLDC:R_1206_3216Metric_Pad1.30x1.75mm_HandSolder
- RBEM_A1, RBEM_B1, RBEM_C1, Rdiv2: value ~ -> 3.3k 1%; footprint Resistor_SMD:R_2512_6332Metric_Pad1.40x3.35mm_HandSolder -> ESC_BLDC:R_1206_3216Metric_Pad1.30x1.75mm_HandSolder
- RBEM_A2, RBEM_B2, RBEM_C2: value ~ -> 39k 1%; footprint Resistor_SMD:R_2512_6332Metric_Pad1.40x3.35mm_HandSolder -> ESC_BLDC:R_1206_3216Metric_Pad1.30x1.75mm_HandSolder
- RBEM_REF_A1: renamed from CBEM_REF_A1; value ~ -> 1k; footprint Capacitor_SMD:C_1206_3216Metric_Pad1.33x1.80mm_HandSolder -> ESC_BLDC:R_1206_3216Metric_Pad1.30x1.75mm_HandSolder; symbol Device:C -> Device:R
- RBEM_REF_B1: renamed from CBEM_REF_B1; value ~ -> 1k; footprint Capacitor_SMD:C_1206_3216Metric_Pad1.33x1.80mm_HandSolder -> ESC_BLDC:R_1206_3216Metric_Pad1.30x1.75mm_HandSolder; symbol Device:C -> Device:R
- RBEM_REF_C1: renamed from CBEM_REF_C1; value ~ -> 1k; footprint Capacitor_SMD:C_1206_3216Metric_Pad1.33x1.80mm_HandSolder -> ESC_BLDC:R_1206_3216Metric_Pad1.30x1.75mm_HandSolder; symbol Device:C -> Device:R
- RBUFIN+1, RBUFIN+2, RBUFIN+3, RBUFIN+4, RBUFIN+5, RBUFIN+6: value ~ -> 1k; footprint Resistor_SMD:R_2512_6332Metric_Pad1.40x3.35mm_HandSolder -> ESC_BLDC:R_1206_3216Metric_Pad1.30x1.75mm_HandSolder
- RBUFIN-1, RBUFIN-2, RBUFIN-3, RBUFIN-4, RBUFIN-5: value ~ -> 100k 1%; footprint Resistor_SMD:R_2512_6332Metric_Pad1.40x3.35mm_HandSolder -> ESC_BLDC:R_1206_3216Metric_Pad1.30x1.75mm_HandSolder
- RBUFIN-6: renamed from RIB1; value ~ -> 100k 1%; footprint Resistor_SMD:R_2512_6332Metric_Pad1.40x3.35mm_HandSolder -> ESC_BLDC:R_1206_3216Metric_Pad1.30x1.75mm_HandSolder
- RBUFOUT1, RBUFOUT2, RBUFOUT3, RBUFOUT4, RBUFOUT5, RBUFOUT6, RNEU_A1, RNEU_B1, RNEU_C1: value ~ -> 10k 1%; footprint Resistor_SMD:R_2512_6332Metric_Pad1.40x3.35mm_HandSolder -> ESC_BLDC:R_1206_3216Metric_Pad1.30x1.75mm_HandSolder
- RIA1, RIC1: value ~ -> 10m 1% 1W; footprint Resistor_SMD:R_2512_6332Metric_Pad1.40x3.35mm_HandSolder -> ESC_BLDC:R_2512_6332Metric_Pad1.40x3.35mm_HandSolder
- RIB1: renamed from RIB2; value ~ -> 10m 1% 1W; footprint Resistor_SMD:R_2512_6332Metric_Pad1.40x3.35mm_HandSolder -> ESC_BLDC:R_2512_6332Metric_Pad1.40x3.35mm_HandSolder
- RPOT1: value R_Pot1 -> 10k lin (extern); footprint TerminalBlock:TerminalBlock_bornier-3_P5.08mm -> ESC_BLDC:TerminalBlock_bornier-3_P5.08mm
- RPull1, RPull2, RPull3: value ~ -> 4.7k; footprint Resistor_SMD:R_2512_6332Metric_Pad1.40x3.35mm_HandSolder -> ESC_BLDC:R_1206_3216Metric_Pad1.30x1.75mm_HandSolder
- Rdiv1: value ~ -> 35.7k 1%; footprint Resistor_SMD:R_2512_6332Metric_Pad1.40x3.35mm_HandSolder -> ESC_BLDC:R_1206_3216Metric_Pad1.30x1.75mm_HandSolder
- U1, U2: footprint (none) -> ESC_BLDC:SOIC-14_3.9x8.7mm_P1.27mm
- U3: footprint LMS8117AMP-3.3/NOPB:MP04A -> ESC_BLDC:SOT-223
- U4: footprint LM339DR:D14 -> ESC_BLDC:SOIC-14_3.9x8.7mm_P1.27mm
- U5: footprint TM4C123GXL:MODULE_EK-TM4C123GXL -> ESC_BLDC:MODULE_EK-TM4C123GXL
- U6, U7, U8: footprint IR2301SPBF:SOIC8L_INF -> ESC_BLDC:SOIC-8_3.9x4.9mm_P1.27mm
Connections:
- net GND: now also CADES2.2, CBDES2.2, CCDES2.2, U4.11 (4IN+), CAHF1.2, CBHF1.2, CCHF1.2, C_U1.2, C_U2.2, C_U4.2, J_SPI.5 (Pin_5), TP_GND1.1 (Pin_1), TP_GND2.1 (Pin_1), TP_GND3.1 (Pin_1), U2.10 (+), U2.12 (+); no longer CADES2.1, CBDES2.1, CCDES2.1
- net OpC1: no longer J7.6 (Pin_6), RBUFIN-6.2, RBUFOUT6.1, U2.6 (-)
- net VCC: now also CADES2.1, CBDES2.1, CCDES2.1, CAHF1.1, CBHF1.1, CCHF1.1; no longer CADES2.2, CBDES2.2, CCDES2.2
- net SPI_MOSI: now reaches U5.J1_8 (PA5)
- net SPI_MOSI: now also J_SPI.4 (Pin_4)
- net SPI_CLK: now reaches U5.J2_10 (PA2)
- net SPI_CLK: now also J_SPI.1 (Pin_1)
- net SPI_MISO: now reaches U5.J2_8 (PA4)
- net SPI_MISO: now also J_SPI.3 (Pin_3)
- net SPI_CS: now reaches U5.J2_9 (PA3)
- net SPI_CS: now also J_SPI.2 (Pin_2)
- net +3V3: now reaches U3.4 (Vout)
- net +3V3: now also CDES2.1, CDESPOT1.1, CPOT5.1, J11.1 (Pin_1), RPOT1.1, RPull1.2, RPull2.2, RPull3.2, U1.4 (V+), U2.4 (V+), U3.2 (Vout), U4.10 (4IN-), U4.3 (VCC), U5.J1_1 (+3.3V), C_U1.1, C_U2.1, C_U4.1
- removed net 3.3V: CDES2.1, CDESPOT1.1, CPOT5.1, J11.1 (Pin_1), RPOT1.1, RPull1.2, RPull2.2, RPull3.2, U1.4 (V+), U2.4 (V+), U3.3 (Vin), U4.3 (VCC), U5.J1_1 (+3.3V)
- net 5V renamed +5V
- net +5V: now also U3.3 (Vin); no longer U3.2 (Vout)
- new net: U2.13 (-), U2.14
- new net: U2.8, U2.9 (-)
- new net OpC2: J7.6 (Pin_6), RBUFIN-6.2, RBUFOUT6.1, U2.6 (-)
- no-connect marks 6 -> 22
Other:
- note added: "1N4149: pics de carrega de Cboot < 1 us (IFSM 4 A @1 us); mitjana ~mA. OK."
- note added: "1N5819: Schottky 40 V / 1 A > 12 V i Io<0.3 A. OK."
- note added: "Afegits TP_GND1..3 + TP de +3V3, +5V i VCC repartits per la placa."
- note added: "C_U1/C_U2: LM324 (pin 4) C_U4: LM339 (pin 3) al costat de cada IC"
- note added: "Cin LDO 10 uF ceramica; Cout 10 uF TANTAL (ESR 0.5-5 ohm, estabilitat LMS8117A)."
- note added: "CxHF1: HF al drenador del MOSFET high-side de cada fase"
- note added: "DESACOBLAMENT, CONNECTOR SPI (LSE2) I TEST POINTS GND"
- note added: "Diode Vout->Vin LDO: no cal (Cout=10 uF << 1000 uF, datasheet LMS8117A)."
- note added: "FB = sensat de la sortida: a la versio fixa de 5 V va directament a +5V (sense divisor)."
- note added: "I_LED = (12-2)/1k = 10 mA"
- note added: "L: AP1509 150 kHz, 12->5 V: dI=(Vin-Vo)D/(fL) -> 39 uH dona 0.5 App (4.7 uH donava 4.1 App!)."
- note added: "NOTES DE DISSENY (valors verificats) VCC = 12 V. Buck AP1509-50 -> +5V; LDO LMS8117-3.3 -> +3V3 (alimenta la LaunchPad pel pin +3.3V). Driver: R_in=33R + 100 pF (tau=3.3 ns); Rg=33R -> t_on~Qg/Io+=325 ns, t_off~186 ns. Cboot=1 uF X7R: dV=(Qg+Iqbs*t)/C = 0.31 V per 2.4 ms (fase OL mes llarga). Cboot ceramic, no electrolitic. Shunt 10 mohm 2512: 0.25 W @5 A. Divisor BEMF 39k/3.3k = 0.078 -> 0.94 V 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"
- note added: "Opamps: buffers (G=1.1) que aillen els divisors d alta impedancia dels comparadors i del filtre."
- note added: "PWR_FLAG (ERC): VCC/GND entren per J_DC1 (pins passius); +3V3 surt d un pin output del LDO; VBx i FASE_x alimenten els pins power_in VB/VS dels IR2301"
- note added: "SSI0: PA2=CLK, PA3=FSS, PA4=RX(MISO), PA5=TX(MOSI)"
- note added: "U2C/U2D no usats: seguidors amb IN+ a GND"
- note removed: "30mA typ current"
- note removed: "Cal diode de proteccio en inversa?"
- note removed: "Calcular L"
- note removed: "Capacitats a prop del LDO i ceramiques"
- note removed: "Diode pasen mes de 500mA??"
- note removed: "FB es nomes output?"
- note removed: "comprobar q model del diode es bo per aquest sistema"
- note removed: "considerar posar mes tp d'alimentacio en varis llocs de la placa"
- note removed: "pq fa falta opamp?"
