File: Controlador_BLDC/Controlador_BLDC.kicad_sch (KiCad schematic)
At the start: 14 parts, among them U1 EK-TM4C123GXL, U2 IR2301SPBF

Commit message: Kicad despres de classe
Parts:
- removed CABO2: ~, Capacitor_SMD:C_1206_3216Metric_Pad1.33x1.80mm_HandSolder, symbol Device:C
- added CADES1, CBDES1, CBH, CBH1, CBH2, CBH3, CBH4, CBH5, CBH6, CBH7, CBH8, CBH9, CBL, CCDES1, CCH, CCL: ~, Capacitor_SMD:C_1206_3216Metric_Pad1.33x1.80mm_HandSolder, symbol Device:C
- added CA_BOOT, CBDES2, CB_BOOT, CCDES2, CC_BOOT: ~, Capacitor_SMD:C_Elec_6.3x5.8, symbol Device:C
- added CDES1: ~, Capacitor_THT:C_Radial_D12.5mm_H20.0mm_P5.00mm, symbol Device:C
- added D1, D2: 1N4149, Diode_THT:D_DO-35_SOD27_P7.62mm_Horizontal, symbol Diode:1N4149
- added D4: 1N5819, Diode_THT:D_DO-41_SOD81_P10.16mm_Horizontal, symbol Diode:1N5819
- added D5: ~, LED_THT:LED_D3.0mm, symbol Device:LED
- added J_DC1: ~, TerminalBlock_Phoenix:TerminalBlock_Phoenix_MKDS-1,5-2-5.08_1x02_P5.08mm_Horizontal, symbol Connector:Screw_Terminal_01x02
- added MOSFET3, MOSFET4, MOSFET5, MOSFET6: IRFR1205TRPBF, D-PAK_TO-252AA_INF, symbol IRFR1205TRPBF:IRFR1205TRPBF
- added R1, RBH, RBL, RCH, RCL, RGBH, RGBL, RGCH, RGCL: ~, Resistor_SMD:R_1206_3216Metric_Pad1.30x1.75mm_HandSolder, symbol Device:R
- added RIB, RIB1, RIB10, RIB11, RIB2, RIB3, RIB4, RIB5, RIB6, RIB7, RIB8, RIB9, RIC: ~, Resistor_SMD:R_2512_6332Metric_Pad1.40x3.35mm_HandSolder, symbol Device:R
- added U2, U3: IR2301SPBF, SOIC8L_INF, symbol IR2301SPBF:IR2301SPBF
- added U4: LMS8117AMP-3.3/NOPB, MP04A, symbol LMS8117AMP-3.3/NOPB:LMS8117AMP-3.3_NOPB
- D3: value ~ -> 1N4149
- renumbered CAHI2 to CAH2, CAHLI1 to CAL, RAHI2 to RAH, RAHI3 to RAL, RGAH2 to RGAH, RGAL2 to RGAL, RIA2 to RIA, U2 to U1
Connections:
- net A: now also CA_BOOT.1, CC_BOOT.1, MOSFET5.3 (S), MOSFET6.2 (D), U3.6 (VS)
- net GND: now also CADES1.1, CBDES1.1, CBDES2.1, CBH.1, CBH2.2, CBH4.2, CBH6.2, CBH7.2, CBH8.1, CBH9.1, CBL.2, CCDES1.1, CCDES2.1, CCH.1, CCL.2, CDES1.2, J_DC1.2 (Pin_2), R1.2, RIB.2, RIB1.2, RIB11.2, RIB2.2, RIB3.2, RIC.2, U2.4 (COM), U3.4 (COM), U4.1 (ADJ/GND)
- net VCC: now also CADES1.2, CBDES1.2, CBDES2.2, CCDES1.2, CCDES2.2, CDES1.1, D1.2 (A), D2.2 (A), D5.2 (A), J_DC1.1 (Pin_1), MOSFET3.2 (D), MOSFET5.2 (D), U2.1 (VCC), U3.1 (VCC)
- net at U1.8 (VB): now also CA_BOOT.2, D1.1 (K); no longer D3.1 (K)
- net AH: now reaches RAH.2
- net AH: now also RBH.2, RCH.2
- net 3.3V: now reaches U1.J1_1 (+3.3V)
- net 3.3V: now also U1.J1_3 (PB0), CBH9.2, U4.2 (Vout)
- net 5V: now reaches U1.J3_1 (+VBUS)
- net AL: now reaches RAL.2
- net AL: now also RBL.2, RCL.2
- new net: CBH.2, RBH.1, U2.2 (HIN)
- new net: CC_BOOT.2, D3.1 (K), U3.8 (VB)
- new net: CBH1.1, CBH2.1, RIB1.1, RIB4.1
- new net: MOSFET4.1 (G), RGBL.1
- new net: RGBL.2, U2.5 (LO)
- new net: CBH3.1, CBH4.1, RIB2.1, RIB5.1
- new net: D5.1 (K), R1.1
- new net: CBH5.1, CBH6.1, RIB3.1, RIB6.1
- new net: CCH.2, RCH.1, U3.2 (HIN)
- new net: CBH8.2, U4.3 (Vin)
- new net: RIB6.2, RIB9.1
- new net: CBL.1, RBL.1, U2.3 (LIN)
- new net: RGBH.2, U2.7 (HO)
- new net: CB_BOOT.2, D2.1 (K), U2.8 (VB)
- new net: MOSFET4.3 (S), RIB.1
- new net: RIB10.1, RIB7.2, RIB8.2, RIB9.2
- new net: MOSFET6.3 (S), RIC.1
- new net: CBH7.1, RIB10.2, RIB11.1
- new net: MOSFET3.1 (G), RGBH.1
- new net: MOSFET6.1 (G), RGCL.1
- new net: MOSFET5.1 (G), RGCH.1
- new net: RIB4.2, RIB7.1
- new net: RIB5.2, RIB8.1
- new net: CCL.1, RCL.1, U3.3 (LIN)
- new net: RGCL.2, U3.5 (LO)
- new net: RGCH.2, U3.7 (HO)
- new net B: CB_BOOT.1, MOSFET3.3 (S), MOSFET4.2 (D), U2.6 (VS)
Other:
- note added: "ALIMENTACIÓ FONT 12 V"
- note added: "Driver A"
- note added: "Driver B"
- note added: "Driver C"
- note added: "Driver de 3 fases"
- note added: "Microcontrolador"
- moved on the sheet: CADES2, CAH2, CAL, MOSFET1, MOSFET2, RAH, RAL, RGAH, RGAL, RIA, U1

Commit message: Entrada de potencia, noves petjades
Parts:
- removed CBH8, CBH9: ~, Capacitor_SMD:C_1206_3216Metric_Pad1.33x1.80mm_HandSolder, symbol Device:C
- removed U4: LMS8117AMP-3.3/NOPB, MP04A, symbol LMS8117AMP-3.3/NOPB:LMS8117AMP-3.3_NOPB
- added CDES, CDES5V2, CPOT1: ~, Capacitor_SMD:C_1206_3216Metric_Pad1.33x1.80mm_HandSolder, symbol Device:C
- added IC1: AP63201WU-7, SOT95P280X100-6N, symbol AP63201WU-7:AP63201WU-7
- added J1: Conn_01x03, symbol Connector_Generic:Conn_01x03
- added L1: SRN4018-4R7M, IND_BOURNS_SRN4018, symbol SRN4018-4R7M:SRN4018-4R7M
- added RPOT1: R_Pot1, Library_modifications_pontH:Potentiometer_Alps_RK163_Single_Horizontal_modified, symbol Device:R_Potentiometer
- added U1: TLV76150DCY, Package_TO_SOT_SMD:SOT-223-3_TabPin2, symbol Regulator_Linear:TLV76150DCY
- U2: renamed from U1; footprint EK-TM4C123GXL:MODULE_EK-TM4C123GXL -> TM4C123GXL:MODULE_EK-TM4C123GXL
- renumbered CAH2 to CAH1, CAL to CAL1, CA_BOOT to CA_BOOT1, CBH to CBH10, CBH4 to CBH5, CBH5 to CBH6, CBH6 to CBH7, CBH7 to CBH8, CBL to CBL1, CB_BOOT to CB_BOOT1, CCH to CCH1, CCL to CCL1, CC_BOOT to CC_BOOT1, D5 to D1, D4 to D2, D1 to D3, D2 to D4, D3 to D5, RAH to RAH1, RAL to RAL1, RBH to RBH1, RBL to RBL1, RCH to RCH1, RCL to RCL1, RGAH to RGAH1, RGAL to RGAL1, RGBH to RGBH1, RGBL to RGBL1, RGCH to RGCH1, RGCL to RGCL1, RIA to RIA1, RIB to RIB12, RIB4 to RIB2, RIB7 to RIB3, RIB2 to RIB4, RIB8 to RIB6, RIB3 to RIB7, RIB6 to RIB8, RIC to RIC1, U1 to U3, U2 to U4, U3 to U5
Connections:
- net 3.3V: no longer U2.J1_3 (PB0)
- net 5V: now also CDES.1, CDES5V2.1, RPOT1.1
- net AH: now also U2.J1_9 (PA6); no longer RBH1.2
- net AL: now also U2.J1_5 (PE4); no longer RBL1.2
- net GND: now also CDES.2, CDES5V2.2, CPOT1.2, RPOT1.3
- net BH: now reaches U2.J1_10 (PA7)
- net BL: now reaches U2.J1_6 (PE5)
- net CL: now reaches U2.J1_7 (PB4)
- net CL: now also RBL1.2
- net CH: now reaches U2.J3_10 (PF1)
- net CH: now also RBH1.2
- new net DUTY: CPOT1.1, RPOT1.2
Other:
- note added: "CONSIGNA MOTOR"

Commit message: Esquematic semi acabat
Falta els valors de resistencies de calcul BEMF, ja que no son E6. S'ha: colocat la petjada a tots els components, arreglat els errors de ERC, calculat valors de L, C i diode de shotkky pel BUCK, solucionat error de footprints del ldo, nous models importats en el segënt commit
Parts:
- removed D1: ~, LED_THT:LED_D3.0mm, symbol Device:LED
- removed D2: 1N5819, Diode_THT:D_DO-41_SOD81_P10.16mm_Horizontal, symbol Diode:1N5819
- removed IC1: AP63201WU-7, SOT95P280X100-6N, symbol AP63201WU-7:AP63201WU-7
- removed L1: SRN4018-4R7M, IND_BOURNS_SRN4018, symbol SRN4018-4R7M:SRN4018-4R7M
- removed RIB10, RIB11: ~, Resistor_SMD:R_2512_6332Metric_Pad1.40x3.35mm_HandSolder, symbol Device:R
- removed U1: TLV76150DCY, Package_TO_SOT_SMD:SOT-223-3_TabPin2, symbol Regulator_Linear:TLV76150DCY
- removed U3, U4: IR2301SPBF, SOIC8L_INF, symbol IR2301SPBF:IR2301SPBF
- added CBUCKDESI1, C_U1, C_U2: 100nF, Capacitor_SMD:C_1206_3216Metric_Pad1.33x1.80mm_HandSolder, symbol Device:C
- added CBUCKDESI2: 10uF, Capacitor_SMD:C_1206_3216Metric_Pad1.33x1.80mm_HandSolder, symbol Device:C
- added CBUCKDESO1: 470uF, Capacitor_SMD:CP_Elec_10x10.5, symbol Device:C_Polarized
- added CDiv1: 22nF 5%, Capacitor_SMD:C_1206_3216Metric_Pad1.33x1.80mm_HandSolder, symbol Device:C
- added CPOT1, CPOT3: 10uF, Capacitor_Tantalum_SMD:CP_EIA-2012-12_Kemet-R, symbol Device:C_Polarized
- added CbypassB1, CbypassC1: 100pF, Capacitor_SMD:C_1206_3216Metric_Pad1.33x1.80mm_HandSolder, symbol Device:C
- added D1: B240A-13-F, B240A-13-F:DIOM5226X230N, symbol B240A-13-F:B240A-13-F
- added IC1: AP1509-50SG-13, AP1509-50SG-13:SOIC127P600X170-8N, symbol AP1509-50SG-13:AP1509-50SG-13
- added IC2: LMS8117AMP-3.3_NOPB, LMS8117AMP-3.3/NOPB:SOT230P700X180-4N, symbol LMS8117AMP-3.3/NOPB:LMS8117AMP-3.3_NOPB
- added J1: Conn_01x05, Connector_PinHeader_2.54mm:PinHeader_1x05_P2.54mm_Vertical, symbol Connector_Generic:Conn_01x05
- added J10: TP_DUTY, Connector_PinHeader_2.54mm:PinHeader_1x02_P2.54mm_Vertical, symbol Connector:Conn_01x02_Pin
- added J11: TP_BUCK, Connector:FanPinHeader_1x04_P2.54mm_Vertical, symbol Connector:Conn_01x04_Pin
- added J12: TP_+3V3, Connector_PinHeader_2.54mm:PinHeader_1x02_P2.54mm_Vertical, symbol Connector:Conn_01x02_Pin
- added J13: TP_+5V, Connector_PinHeader_2.54mm:PinHeader_1x02_P2.54mm_Vertical, symbol Connector:Conn_01x02_Pin
- added J14: TP_VCC, Connector_PinHeader_2.54mm:PinHeader_1x02_P2.54mm_Vertical, symbol Connector:Conn_01x02_Pin
- added J3: TP_SENSOR, Connector_PinHeader_2.54mm:PinHeader_1x04_P2.54mm_Vertical, symbol Connector:Conn_01x04_Pin
- added J4: TP_BEMF, Connector_PinHeader_2.54mm:PinHeader_1x04_P2.54mm_Vertical, symbol Connector:Conn_01x04_Pin
- added J5: TP_VREF_ADC, Connector_PinHeader_2.54mm:PinHeader_1x04_P2.54mm_Vertical, symbol Connector:Conn_01x04_Pin
- added J6: TP_VNDIV, Connector_PinHeader_2.54mm:PinHeader_1x04_P2.54mm_Vertical, symbol Connector:Conn_01x04_Pin
- added J7: TP_BEMFD, Connector_PinHeader_2.54mm:PinHeader_1x04_P2.54mm_Vertical, symbol Connector:Conn_01x04_Pin
- added J8: TP_OPAMP, Connector_PinHeader_2.54mm:PinHeader_1x07_P2.54mm_Vertical, symbol Connector:Conn_01x07_Pin
- added J9: TP_NEUTRE, Connector_PinHeader_2.54mm:PinHeader_1x02_P2.54mm_Vertical, symbol Connector:Conn_01x02_Pin
- added J_TPA1: TP_FASE_A, Connector_PinHeader_2.54mm:PinHeader_1x05_P2.54mm_Vertical, symbol Connector:Conn_01x05_Pin
- added J_TPA2: TP_FASE_B, Connector_PinHeader_2.54mm:PinHeader_1x05_P2.54mm_Vertical, symbol Connector:Conn_01x05_Pin
- added J_TPA3: TP_FASE_C, Connector_PinHeader_2.54mm:PinHeader_1x05_P2.54mm_Vertical, symbol Connector:Conn_01x05_Pin
- added J_VBA1: TP_VBA, Connector_PinHeader_2.54mm:PinHeader_1x01_P2.54mm_Vertical, symbol Connector:Conn_01x01_Pin
- added J_VBA2: TP_VBB, Connector_PinHeader_2.54mm:PinHeader_1x01_P2.54mm_Vertical, symbol Connector:Conn_01x01_Pin
- added J_VBA3: TP_VBC, Connector_PinHeader_2.54mm:PinHeader_1x01_P2.54mm_Vertical, symbol Connector:Conn_01x01_Pin
- added J_VBA4: TP_FASE_A, Connector_PinHeader_2.54mm:PinHeader_1x01_P2.54mm_Vertical, symbol Connector:Conn_01x01_Pin
- added J_VBA5: TP_FASE_B, Connector_PinHeader_2.54mm:PinHeader_1x01_P2.54mm_Vertical, symbol Connector:Conn_01x01_Pin
- added J_VBA6: TP_FASE_C, Connector_PinHeader_2.54mm:PinHeader_1x01_P2.54mm_Vertical, symbol Connector:Conn_01x01_Pin
- added L1: CDRH127_LDNP-470MC, CDRH127-LDNP-470MC:INDPM120120X800N, symbol CDRH127-LDNP-470MC:CDRH127_LDNP-470MC
- added LED1: LTL-4221N (vermell), LIB_LTL-4221N:LTL4221N, symbol LIB_LTL-4221N:LTL-4221N
- added RBUFIN+1, RBUFIN+2, RBUFIN+3, RBUFIN+4, RBUFIN+5, RBUFIN+6: 1k, Resistor_SMD:R_1206_3216Metric_Pad1.30x1.75mm_HandSolder, symbol Device:R
- added RBUFIN-1, RBUFIN-2, RBUFIN-3, RBUFIN-4, RBUFIN-5, RBUFIN-6: 100k 1%, Resistor_SMD:R_1206_3216Metric_Pad1.30x1.75mm_HandSolder, symbol Device:R
- added RBUFOUT1, RBUFOUT2, RBUFOUT3, RBUFOUT4, RBUFOUT5, RBUFOUT6: 10k 1%, Resistor_SMD:R_1206_3216Metric_Pad1.30x1.75mm_HandSolder, symbol Device:R
- added RPull1, RPull2, RPull3: 4.7k, Resistor_SMD:R_1206_3216Metric_Pad1.30x1.75mm_HandSolder, symbol Device:R
- added Rdiv1: 35.7k 1%, Resistor_SMD:R_1206_3216Metric_Pad1.30x1.75mm_HandSolder, symbol Device:R
- added Rdiv2: 3.3k 1%, Resistor_SMD:R_1206_3216Metric_Pad1.30x1.75mm_HandSolder, symbol Device:R
- added U1, U2: LM324, Package_SO:SOIC-14_3.9x8.7mm_P1.27mm, symbol Amplifier_Operational:LM324
- added U3: LM339DR, LM339DR:D14, symbol LM339DR:LM339DR
- added U6, U7: IR2301SPBF, IR2301SPBF:SOIC8L_INF, symbol IR2301SPBF:IR2301SPBF
- CADES1, CBDES1, CCDES1: value ~ -> 10uF
- CADES2, CBDES2, CCDES2: value ~ -> 100nF; footprint Capacitor_SMD:C_Elec_6.3x5.8 -> Capacitor_SMD:C_1206_3216Metric_Pad1.33x1.80mm_HandSolder
- CAH1, CAL1, CBL1, CCH1, CCL1: value ~ -> 100pF
- CA_BOOT1, CB_BOOT1, CC_BOOT1: value ~ -> 1uF; footprint Capacitor_SMD:C_Elec_6.3x5.8 -> Capacitor_SMD:C_1206_3216Metric_Pad1.33x1.80mm_HandSolder
- CBEM_A1: renamed from CBH2; value ~ -> 22nF 5%
- CBEM_B1: renamed from CBH5; value ~ -> 22nF 5%
- CBEM_C1: renamed from CBH7; value ~ -> 22nF 5%
- CBH1: renamed from CBH10; value ~ -> 100pF
- CDES1: value ~ -> 470uF; footprint Capacitor_THT:C_Radial_D12.5mm_H20.0mm_P5.00mm -> Capacitor_SMD:CP_Elec_10x10.5; symbol Device:C -> Device:C_Polarized
- CDES2: renamed from CDES; value ~ -> 10uF
- CDESPOT1: renamed from CDES5V2; value ~ -> 100nF
- CPOT2: renamed from CPOT1; value ~ -> 100nF
- CbypassA1: renamed from CBH8; value ~ -> 100pF
- D2: renamed from D3; footprint Diode_THT:D_DO-35_SOD27_P7.62mm_Horizontal -> Diode_THT:D_DO-35_SOD27_P10.16mm_Horizontal
- D3: renamed from D4; footprint Diode_THT:D_DO-35_SOD27_P7.62mm_Horizontal -> Diode_THT:D_DO-35_SOD27_P10.16mm_Horizontal
- D4: renamed from D5; footprint Diode_THT:D_DO-35_SOD27_P7.62mm_Horizontal -> Diode_THT:D_DO-35_SOD27_P10.16mm_Horizontal
- J2: renamed from J1; value Conn_01x03 -> MOTOR; footprint (none) -> TerminalBlock_Phoenix:TerminalBlock_Phoenix_MKDS-1,5-3-5.08_1x03_P5.08mm_Horizontal
- J_DC1: value ~ -> 12V_IN; footprint TerminalBlock_Phoenix:TerminalBlock_Phoenix_MKDS-1,5-2-5.08_1x02_P5.08mm_Horizontal -> TerminalBlock:TerminalBlock_bornier-2_P5.08mm
- MOSFET1, MOSFET2, MOSFET3, MOSFET4, MOSFET5, MOSFET6: footprint D-PAK_TO-252AA_INF -> IRFR1205TRPBF:D-PAK_TO-252AA_INF
- R1: value ~ -> 1k
- RAH1, RAL1, RBH1, RBL1, RCH1, RCL1, RGAH1, RGAL1, RGBH1, RGBL1, RGCH1, RGCL1: value ~ -> 33
- RBEM_A1: renamed from RIB1; value ~ -> 3.3k 1%; footprint Resistor_SMD:R_2512_6332Metric_Pad1.40x3.35mm_HandSolder -> Resistor_SMD:R_1206_3216Metric_Pad1.30x1.75mm_HandSolder
- RBEM_A2: renamed from RIB2; value ~ -> 39k 1%; footprint Resistor_SMD:R_2512_6332Metric_Pad1.40x3.35mm_HandSolder -> Resistor_SMD:R_1206_3216Metric_Pad1.30x1.75mm_HandSolder
- RBEM_B1: renamed from RIB4; value ~ -> 3.3k 1%; footprint Resistor_SMD:R_2512_6332Metric_Pad1.40x3.35mm_HandSolder -> Resistor_SMD:R_1206_3216Metric_Pad1.30x1.75mm_HandSolder
- RBEM_B2: renamed from RIB5; value ~ -> 39k 1%; footprint Resistor_SMD:R_2512_6332Metric_Pad1.40x3.35mm_HandSolder -> Resistor_SMD:R_1206_3216Metric_Pad1.30x1.75mm_HandSolder
- RBEM_C1: renamed from RIB7; value ~ -> 3.3k 1%; footprint Resistor_SMD:R_2512_6332Metric_Pad1.40x3.35mm_HandSolder -> Resistor_SMD:R_1206_3216Metric_Pad1.30x1.75mm_HandSolder
- RBEM_C2: renamed from RIB8; value ~ -> 39k 1%; footprint Resistor_SMD:R_2512_6332Metric_Pad1.40x3.35mm_HandSolder -> Resistor_SMD:R_1206_3216Metric_Pad1.30x1.75mm_HandSolder
- RBEM_REF_A1: renamed from CBH1; value ~ -> 1k; footprint Capacitor_SMD:C_1206_3216Metric_Pad1.33x1.80mm_HandSolder -> Resistor_SMD:R_1206_3216Metric_Pad1.30x1.75mm_HandSolder; symbol Device:C -> Device:R
- RBEM_REF_B1: renamed from CBH3; value ~ -> 1k; footprint Capacitor_SMD:C_1206_3216Metric_Pad1.33x1.80mm_HandSolder -> Resistor_SMD:R_1206_3216Metric_Pad1.30x1.75mm_HandSolder; symbol Device:C -> Device:R
- RBEM_REF_C1: renamed from CBH6; value ~ -> 1k; footprint Capacitor_SMD:C_1206_3216Metric_Pad1.33x1.80mm_HandSolder -> Resistor_SMD:R_1206_3216Metric_Pad1.30x1.75mm_HandSolder; symbol Device:C -> Device:R
- RIA1, RIC1: value ~ -> 1m; footprint Resistor_SMD:R_2512_6332Metric_Pad1.40x3.35mm_HandSolder -> Resistor_SMD:R_1206_3216Metric_Pad1.30x1.75mm_HandSolder
- RIB1: renamed from RIB12; value ~ -> 1m; footprint Resistor_SMD:R_2512_6332Metric_Pad1.40x3.35mm_HandSolder -> Resistor_SMD:R_1206_3216Metric_Pad1.30x1.75mm_HandSolder
- RNEU_A1: renamed from RIB3; value ~ -> 10k 1%; footprint Resistor_SMD:R_2512_6332Metric_Pad1.40x3.35mm_HandSolder -> Resistor_SMD:R_1206_3216Metric_Pad1.30x1.75mm_HandSolder
- RNEU_B1: renamed from RIB6; value ~ -> 10k 1%; footprint Resistor_SMD:R_2512_6332Metric_Pad1.40x3.35mm_HandSolder -> Resistor_SMD:R_1206_3216Metric_Pad1.30x1.75mm_HandSolder
- RNEU_C1: renamed from RIB9; value ~ -> 10k 1%; footprint Resistor_SMD:R_2512_6332Metric_Pad1.40x3.35mm_HandSolder -> Resistor_SMD:R_1206_3216Metric_Pad1.30x1.75mm_HandSolder
- RPOT1: value R_Pot1 -> 10k; footprint Library_modifications_pontH:Potentiometer_Alps_RK163_Single_Horizontal_modified -> TerminalBlock:TerminalBlock_bornier-3_P5.08mm
- U5: footprint SOIC8L_INF -> IR2301SPBF:SOIC8L_INF
- renumbered U2 to U4
Connections:
- net B is gone; now on net FASE_B: CB_BOOT1.1, MOSFET3.3 (S), MOSFET4.2 (D)
- net AH: now also U4.J1_5 (PE4); no longer RCH1.2, U4.J1_9 (PA6)
- net AL: now also U4.J1_9 (PA6); no longer RCL1.2, U4.J1_5 (PE4)
- net BH: now also RBH1.2, U4.J1_6 (PE5); no longer U4.J1_10 (PA7)
- net BL: now also RBL1.2, U4.J1_10 (PA7); no longer U4.J1_6 (PE5)
- net CH: now also RCH1.2, U4.J1_7 (PB4); no longer RBH1.2, U4.J3_10 (PF1)
- net CL: now also RCL1.2, U4.J3_10 (PF1); no longer RBL1.2, U4.J1_7 (PB4)
- net DUTY: now also U4.J3_3 (PD0), J10.1 (Pin_1)
- net GND: now also CADES2.2, CBDES2.2, CCDES2.2, RPOT1.1, CBUCKDESI1.2, CBUCKDESI2.2, CBUCKDESO1.2, CDiv1.2, CPOT1.2, CPOT3.2, C_U1.2, C_U2.2, D1.2 (A), IC1.4 (SD), IC1.5 (GND_1), IC1.6 (GND_2), IC1.7 (GND_3), IC1.8 (GND_4), IC2.1 (GND), J1.5 (Pin_5), J10.2 (Pin_2), J11.3 (Pin_3), J11.4 (Pin_4), J12.2 (Pin_2), J13.2 (Pin_2), J14.2 (Pin_2), J3.4 (Pin_4), J4.4 (Pin_4), J5.4 (Pin_4), J6.4 (Pin_4), J7.4 (Pin_4), J8.7 (Pin_7), J_TPA1.5 (Pin_5), J_TPA2.5 (Pin_5), J_TPA3.5 (Pin_5), RBUFIN-1.1, RBUFIN-2.1, RBUFIN-3.1, RBUFIN-4.1, RBUFIN-5.1, RBUFIN-6.1, Rdiv2.1, U1.11 (V-), U2.10 (+), U2.11 (V-), U2.12 (+), U3.11 (4IN+), U3.12 (GND), U6.4 (COM), U7.4 (COM); no longer CADES2.1, CBDES2.1, CCDES2.1, CbypassA1.2, RPOT1.3
- net VCC: now also CADES2.1, CBDES2.1, CCDES2.1, CBUCKDESI1.1, CBUCKDESI2.1, IC1.1 (VIN), J14.1 (Pin_1), LED1.2 (A), U6.1 (VCC), U7.1 (VCC); no longer CADES2.2, CBDES2.2, CCDES2.2
- net HinB: now reaches CBH1.2, RBH1.1
- net HinB: now also U6.2 (HIN)
- net HinA: now reaches CAH1.2, RAH1.1
- net HinA: now also U5.2 (HIN)
- net LinA: now reaches CAL1.1, RAL1.1
- net LinA: now also U5.3 (LIN)
- net GLA: now reaches RGAL1.2
- net GLA: now also U5.5 (LO), J_TPA1.3 (Pin_3)
- net GHA: now reaches RGAH1.2
- net GHA: now also U5.7 (HO), J_TPA1.2 (Pin_2)
- net VBA: now reaches CA_BOOT1.2, D2.1 (K)
- net VBA: now also U5.8 (VB), J_VBA1.1 (Pin_1)
- net VBC: now reaches CC_BOOT1.2, D4.1 (K)
- net VBC: now also J_VBA3.1 (Pin_1), U7.8 (VB); no longer U5.8 (VB)
- net A_BEMF: now reaches CBEM_A1.1, RBEM_A1.1, RBEM_A2.1, RBEM_REF_A1.1
- net A_BEMF: now also J4.1 (Pin_1), RBUFIN+1.1
- net FASE_A: now reaches J2.1 (Pin_1)
- net FASE_A: now also CA_BOOT1.1, MOSFET1.3 (S), MOSFET2.2 (D), RBEM_A2.2, RNEU_A1.1, U5.6 (VS), J_TPA1.1 (Pin_1), J_VBA4.1 (Pin_1)
- net FASE_B: now reaches J2.2 (Pin_2)
- net FASE_B: now also RBEM_B2.2, RNEU_B1.1, J_TPA2.1 (Pin_1), J_VBA5.1 (Pin_1), U6.6 (VS)
- net FASE_C: now reaches J2.3 (Pin_3)
- net FASE_C: now also CC_BOOT1.1, MOSFET5.3 (S), MOSFET6.2 (D), RBEM_C2.2, RNEU_C1.1, J_TPA3.1 (Pin_1), J_VBA6.1 (Pin_1), U7.6 (VS)
- net GLB: now reaches RGBL1.2
- net GLB: now also J_TPA2.3 (Pin_3), U6.5 (LO)
- net B_BEMF: now reaches CBEM_B1.1, RBEM_B1.1, RBEM_B2.1, RBEM_REF_B1.1
- net B_BEMF: now also J4.2 (Pin_2), RBUFIN+3.1
- net at R1.1: now also LED1.1 (K)
- net C_BEMF: now reaches CBEM_C1.1, RBEM_C1.1, RBEM_C2.1, RBEM_REF_C1.1
- net C_BEMF: now also J4.3 (Pin_3), RBUFIN+5.1
- net HinC: now reaches CCH1.2, RCH1.1
- net HinC: now also U7.2 (HIN); no longer U5.2 (HIN)
- net LinB: now reaches CBL1.1, RBL1.1
- net LinB: now also U6.3 (LIN)
- net GHB: now reaches RGBH1.2
- net GHB: now also J_TPA2.2 (Pin_2), U6.7 (HO)
- net VBB: now reaches CB_BOOT1.2, D3.1 (K)
- net VBB: now also J_VBA2.1 (Pin_1), U6.8 (VB)
- net I_B: now reaches MOSFET4.3 (S), RIB1.1
- net I_B: now also J_TPA2.4 (Pin_4)
- net I_A: now reaches MOSFET2.3 (S), RIA1.1
- net I_A: now also J_TPA1.4 (Pin_4)
- net Neu: now reaches RNEU_A1.2, RNEU_B1.2, RNEU_C1.2
- net Neu: now also J9.1 (Pin_1), Rdiv1.1
- net SPI_CS: now reaches U4.J1_8 (PA5)
- net SPI_CS: now also J1.2 (Pin_2)
- net SPI_CLK: now reaches U4.J2_10 (PA2)
- net SPI_CLK: now also J1.1 (Pin_1)
- net SPI_MISO: now reaches U4.J2_8 (PA4)
- net SPI_MISO: now also J1.3 (Pin_3)
- net SPI_MOSI: now reaches U4.J2_9 (PA3)
- net SPI_MOSI: now also J1.4 (Pin_4)
- net SensorA: now reaches U4.J3_4 (PD1)
- net SensorA: now also J3.1 (Pin_1), RPull2.1, U3.2 (2OUT)
- net SensorB: now reaches U4.J3_5 (PD2)
- net SensorB: now also J3.2 (Pin_2), RPull1.1, U3.1 (1OUT)
- net SensorC: now reaches U4.J3_6 (PD3)
- net SensorC: now also J3.3 (Pin_3), RPull3.1, U3.14 (OUT3)
- net A_Vref: now reaches U4.J3_7 (PE1)
- net A_Vref: now also RBEM_REF_A1.2, J5.1 (Pin_1)
- net B_Vref: now reaches U4.J3_8 (PE2)
- net B_Vref: now also RBEM_REF_B1.2, J5.2 (Pin_2)
- net C_Vref: now reaches U4.J3_9 (PE3)
- net C_Vref: now also RBEM_REF_C1.2, J5.3 (Pin_3)
- net I_C: now reaches MOSFET6.3 (S), RIC1.1
- net I_C: now also J_TPA3.4 (Pin_4)
- net A_BEMFD: now reaches CbypassA1.1
- net A_BEMFD: now also J7.1 (Pin_1), RBUFOUT1.2, U1.1, U3.4 (2IN-)
- net LinC: now reaches CCL1.1, RCL1.1
- net LinC: now also U7.3 (LIN); no longer U5.3 (LIN)
- net GLC: now reaches RGCL1.2
- net GLC: now also J_TPA3.3 (Pin_3), U7.5 (LO); no longer U5.5 (LO)
- net GHC: now reaches RGCH1.2
- net GHC: now also J_TPA3.2 (Pin_2), U7.7 (HO); no longer U5.7 (HO)
- net 3.3V renamed +3V3
- net +3V3: now also CDES2.1, CDESPOT1.1, RPOT1.3, CPOT3.1, C_U1.1, C_U2.1, IC2.2 (OUTPUT_1), IC2.4 (OUTPUT_2), J12.1 (Pin_1), RPull1.2, RPull2.2, RPull3.2, U1.4 (V+), U2.4 (V+), U3.10 (4IN-), U3.3 (VCC)
- removed net 5V: CDES2.1, CDESPOT1.1, RPOT1.1, U4.J3_1 (+VBUS)
- removed net A: CA_BOOT1.1, CC_BOOT1.1, MOSFET1.3 (S), MOSFET2.2 (D), MOSFET5.3 (S), MOSFET6.2 (D), U5.6 (VS)
- new net: U2.13 (-), U2.14
- new net: RBUFIN+3.2, U1.10 (+)
- new net: RBUFIN+6.2, U2.5 (+)
- new net: RBUFIN+2.2, U1.5 (+)
- new net: RBUFIN+5.2, U2.3 (+)
- new net: RBUFIN+4.2, U1.12 (+)
- new net: U2.8, U2.9 (-)
- new net: RBUFIN+1.2, U1.3 (+)
- new net +5V: CBUCKDESO1.1, CPOT1.1, IC1.3 (FB), IC2.3 (INPUT), J11.2 (Pin_2), J13.1 (Pin_1), L1.1
- new net BUCKO: D1.1 (K), IC1.2 (OUTPUT), J11.1 (Pin_1), L1.2
- new net B_BEMFD: CbypassB1.1, J7.2 (Pin_2), RBUFOUT3.2, U1.8, U3.6 (1IN-)
- new net C_BEMFD: CbypassC1.1, J7.3 (Pin_3), RBUFOUT5.2, U2.1, U3.8 (3IN-)
- new net Neu_div: CDiv1.1, J9.2 (Pin_2), RBUFIN+2.1, RBUFIN+4.1, RBUFIN+6.1, Rdiv1.2, Rdiv2.2
- new net OpA1: J8.1 (Pin_1), RBUFIN-1.2, RBUFOUT1.1, U1.2 (-)
- new net OpA2: J8.2 (Pin_2), RBUFIN-2.2, RBUFOUT2.1, U1.6 (-)
- new net OpB1: J8.3 (Pin_3), RBUFIN-3.2, RBUFOUT3.1, U1.9 (-)
- new net OpB2: J8.4 (Pin_4), RBUFIN-4.2, RBUFOUT4.1, U1.13 (-)
- new net OpC1: J8.5 (Pin_5), RBUFIN-5.2, RBUFOUT5.1, U2.2 (-)
- new net OpC2: J8.6 (Pin_6), RBUFIN-6.2, RBUFOUT6.1, U2.6 (-)
- new net VNdivA: CbypassA1.2, J6.1 (Pin_1), RBUFOUT2.2, U1.7, U3.5 (2IN+)
- new net VNdivB: CbypassB1.2, J6.2 (Pin_2), RBUFOUT4.2, U1.14, U3.7 (1IN+)
- new net VNdivC: CbypassC1.2, J6.3 (Pin_3), RBUFOUT6.2, U2.7, U3.9 (3IN+)
- no-connect marks 0 -> 21
Other:
- note added: "1N4149: pics de carrega de Cboot < 1 us (IFSM 4 A @1 us); mitjana ~mA. OK."
- note added: "BUCK DC/DC"
- note added: "Condensadors de tantal (petjada temporal)"
- note added: "Connector Fases"
- note added: "Connector SPI"
- note added: "Diode Vout->Vin LDO: no cal (Cout=10 uF << 1000 uF, datasheet LMS8117A)."
- note added: "I_LED =10 mA"
- note added: "LDO"
- note added: "NOTES DE DISSENY (valors verificats) VCC = 12 V. Buck AP1509-50 -> +5V; LDO LMS8117-3.3 -> +3V3 (alimenta la LaunchPad pel pin +3.3V). Driver: R_in=33R + 100 pF (tau=3.3 ns); Rg=33R -> t_on~Qg/Io+=325 ns, t_off~186 ns. Cboot=1 uF X7R: dV=(Qg+Iqbs*t)/C = 0.31 V per 2.4 ms (fase OL mes llarga). Cboot ceramic, no electrolitic. Shunt 10 mohm 2512: 0.25 W @5 A. Divisor BEMF 39k/3.3k = 0.078 -> 0.94 V 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"
- note added: "Nomes es poden resistencies E6"
- note added: "Opamps: buffers (G=1.1) que aillen els divisors d alta impedancia dels comparadors i del filtre."
- note added: "Power Flags"
- note added: "Recuperació BEMF"
- note added: "Test Points"
- note added: "U2C/U2D no usats: seguidors amb IN+ a GND"
- note added: "extern"
- note added: "preguntar quina petjada tantal, lm324, capacitat gran"
- moved on the sheet: CADES1, CBDES1, CBEM_A1, CBEM_B1, CBEM_C1, CCDES1, CDES2, CDESPOT1, CPOT2, CbypassA1, J2, J_DC1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

Commit message: Versió final* de la placa
S'ha canviat la recuperacio BEMF del esquematic, testpoints, i s'ha millorat tots els errors de la pcb
Parts:
- removed CBEM_A1, CBEM_B1, CBEM_C1: 22nF 5%, Capacitor_SMD:C_1206_3216Metric_Pad1.33x1.80mm_HandSolder, symbol Device:C
- removed C_U1, C_U2: 100nF, Capacitor_SMD:C_1206_3216Metric_Pad1.33x1.80mm_HandSolder, symbol Device:C
- removed CbypassA1, CbypassB1, CbypassC1: 100pF, Capacitor_SMD:C_1206_3216Metric_Pad1.33x1.80mm_HandSolder, symbol Device:C
- removed J10: TP_DUTY, Connector_PinHeader_2.54mm:PinHeader_1x02_P2.54mm_Vertical, symbol Connector:Conn_01x02_Pin
- removed J11: TP_BUCK, Connector:FanPinHeader_1x04_P2.54mm_Vertical, symbol Connector:Conn_01x04_Pin
- removed J12: TP_+3V3, Connector_PinHeader_2.54mm:PinHeader_1x02_P2.54mm_Vertical, symbol Connector:Conn_01x02_Pin
- removed J13: TP_+5V, Connector_PinHeader_2.54mm:PinHeader_1x02_P2.54mm_Vertical, symbol Connector:Conn_01x02_Pin
- removed J14: TP_VCC, Connector_PinHeader_2.54mm:PinHeader_1x02_P2.54mm_Vertical, symbol Connector:Conn_01x02_Pin
- removed J3: TP_SENSOR, Connector_PinHeader_2.54mm:PinHeader_1x04_P2.54mm_Vertical, symbol Connector:Conn_01x04_Pin
- removed J4: TP_BEMF, Connector_PinHeader_2.54mm:PinHeader_1x04_P2.54mm_Vertical, symbol Connector:Conn_01x04_Pin
- removed J5: TP_VREF_ADC, Connector_PinHeader_2.54mm:PinHeader_1x04_P2.54mm_Vertical, symbol Connector:Conn_01x04_Pin
- removed J6: TP_VNDIV, Connector_PinHeader_2.54mm:PinHeader_1x04_P2.54mm_Vertical, symbol Connector:Conn_01x04_Pin
- removed J7: TP_BEMFD, Connector_PinHeader_2.54mm:PinHeader_1x04_P2.54mm_Vertical, symbol Connector:Conn_01x04_Pin
- removed J8: TP_OPAMP, Connector_PinHeader_2.54mm:PinHeader_1x07_P2.54mm_Vertical, symbol Connector:Conn_01x07_Pin
- removed J9: TP_NEUTRE, Connector_PinHeader_2.54mm:PinHeader_1x02_P2.54mm_Vertical, symbol Connector:Conn_01x02_Pin
- removed J_TPA1: TP_FASE_A, Connector_PinHeader_2.54mm:PinHeader_1x05_P2.54mm_Vertical, symbol Connector:Conn_01x05_Pin
- removed J_TPA2: TP_FASE_B, Connector_PinHeader_2.54mm:PinHeader_1x05_P2.54mm_Vertical, symbol Connector:Conn_01x05_Pin
- removed J_TPA3: TP_FASE_C, Connector_PinHeader_2.54mm:PinHeader_1x05_P2.54mm_Vertical, symbol Connector:Conn_01x05_Pin
- removed J_VBA1: TP_VBA, Connector_PinHeader_2.54mm:PinHeader_1x01_P2.54mm_Vertical, symbol Connector:Conn_01x01_Pin
- removed J_VBA2: TP_VBB, Connector_PinHeader_2.54mm:PinHeader_1x01_P2.54mm_Vertical, symbol Connector:Conn_01x01_Pin
- removed J_VBA3: TP_VBC, Connector_PinHeader_2.54mm:PinHeader_1x01_P2.54mm_Vertical, symbol Connector:Conn_01x01_Pin
- removed J_VBA4: TP_FASE_A, Connector_PinHeader_2.54mm:PinHeader_1x01_P2.54mm_Vertical, symbol Connector:Conn_01x01_Pin
- removed J_VBA5: TP_FASE_B, Connector_PinHeader_2.54mm:PinHeader_1x01_P2.54mm_Vertical, symbol Connector:Conn_01x01_Pin
- removed J_VBA6: TP_FASE_C, Connector_PinHeader_2.54mm:PinHeader_1x01_P2.54mm_Vertical, symbol Connector:Conn_01x01_Pin
- removed RBEM_A1, RBEM_B1, RBEM_C1: 3.3k 1%, Resistor_SMD:R_1206_3216Metric_Pad1.30x1.75mm_HandSolder, symbol Device:R
- removed RBEM_A2, RBEM_B2, RBEM_C2: 39k 1%, Resistor_SMD:R_1206_3216Metric_Pad1.30x1.75mm_HandSolder, symbol Device:R
- removed RBEM_REF_A1, RBEM_REF_B1, RBEM_REF_C1, RBUFIN+1, RBUFIN+2, RBUFIN+3, RBUFIN+4, RBUFIN+5, RBUFIN+6: 1k, Resistor_SMD:R_1206_3216Metric_Pad1.30x1.75mm_HandSolder, symbol Device:R
- removed RBUFIN-1, RBUFIN-2, RBUFIN-3, RBUFIN-4, RBUFIN-5, RBUFIN-6: 100k 1%, Resistor_SMD:R_1206_3216Metric_Pad1.30x1.75mm_HandSolder, symbol Device:R
- removed RBUFOUT1, RBUFOUT2, RBUFOUT3, RBUFOUT4, RBUFOUT5, RBUFOUT6, RNEU_A1, RNEU_B1, RNEU_C1: 10k 1%, Resistor_SMD:R_1206_3216Metric_Pad1.30x1.75mm_HandSolder, symbol Device:R
- removed RIA1, RIB1, RIC1: 1m, Resistor_SMD:R_1206_3216Metric_Pad1.30x1.75mm_HandSolder, symbol Device:R
- removed U1, U2: LM324, Package_SO:SOIC-14_3.9x8.7mm_P1.27mm, symbol Amplifier_Operational:LM324
- removed U3: LM339DR, LM339DR:D14, symbol LM339DR:LM339DR
- added CDESCOMP1: 100nF, Capacitor_SMD:C_1206_3216Metric_Pad1.33x1.80mm_HandSolder, symbol Device:C
- added Cb1, Cb2, Cb3: 33nF, Capacitor_SMD:C_1206_3216Metric_Pad1.33x1.80mm_HandSolder, symbol Device:C
- added Cgnd1, Cgnd2, Cgnd3: 0.1nF, Capacitor_SMD:C_1206_3216Metric_Pad1.33x1.80mm_HandSolder, symbol Device:C
- added H1, H2, H3, H4: MountingHole, MountingHole:MountingHole_4.3mm_M4_ISO14580, symbol Mechanical:MountingHole
- added J_TP1, J_TP2, J_TP3: Conn_01x03_Pin, Connector_PinHeader_2.54mm:PinHeader_1x03_P2.54mm_Vertical, symbol Connector:Conn_01x03_Pin
- added J_TP4, J_TPG1, J_TPG2, J_TPG3: Conn_01x02_Pin, Connector_PinHeader_2.54mm:PinHeader_1x02_P2.54mm_Vertical, symbol Connector:Conn_01x02_Pin
- added J_TP5, J_TPA1, J_TPB1, J_TPC1: Conn_01x04_Pin, Connector_PinHeader_2.54mm:PinHeader_1x04_P2.54mm_Vertical, symbol Connector:Conn_01x04_Pin
- added RdivA1, RdivB1, RdivC1: 10k, Resistor_SMD:R_1206_3216Metric_Pad1.30x1.75mm_HandSolder, symbol Device:R
- added RdivA2, RdivB2, RdivC2: 33k, Resistor_SMD:R_1206_3216Metric_Pad1.30x1.75mm_HandSolder, symbol Device:R
- added Rstar_A1, Rstar_B1, Rstar_C1: 1k, Resistor_SMD:R_1206_3216Metric_Pad1.30x1.75mm_HandSolder, symbol Device:R
- added U1: LM339DR, LM339DR:D14, symbol LM339DR:LM339DR
- CDiv1: value 22nF 5% -> 0.1nF
- D2, D3, D4: footprint Diode_THT:D_DO-35_SOD27_P10.16mm_Horizontal -> Diode_THT:D_DO-35_SOD27_P7.62mm_Horizontal
- Rdiv1: value 35.7k 1% -> 33k
- Rdiv2: value 3.3k 1% -> 10k
- U2: renamed from U4; footprint TM4C123GXL:MODULE_EK-TM4C123GXL -> TIVA-Modfied:MODULE_EK-TM4C123GXL_mofied
- renumbered CBUCKDESI1 to CBD1, CBUCKDESI2 to CBD2, CDESPOT1 to CDP1, CPOT1 to CLDO1, CPOT3 to CLDO2, CPOT2 to CPOT1, U5 to U3, U6 to U4, U7 to U5
Connections:
- net A_Vref is gone; now on net Neu_div: U2.J3_7 (PE1)
- net I_A is gone; now on net GND: MOSFET2.3 (S)
- net I_B is gone; now on net GND: MOSFET4.3 (S)
- net I_C is gone; now on net GND: MOSFET6.3 (S)
- net +3V3: now also J_TP2.2 (Pin_2)
- net +5V: now also CDESCOMP1.1, J_TP1.3 (Pin_3), U1.10 (4IN-), U1.3 (VCC)
- net AH: now also U2.J1_7 (PB4); no longer U2.J1_5 (PE4)
- net AL: now also U2.J3_10 (PF1); no longer U2.J1_9 (PA6)
- net A_BEMF: now also Cb1.1, Cgnd1.1, J_TP4.2 (Pin_2), RdivA1.1, RdivA2.1, U1.4 (2IN-)
- net BUCKO: now also J_TP1.1 (Pin_1)
- net B_BEMF: now also Cb2.1, Cgnd2.1, J_TP3.2 (Pin_2), RdivB1.1, RdivB2.1, U1.6 (1IN-)
- net CH: now also U2.J1_5 (PE4); no longer U2.J1_7 (PB4)
- net CL: now also U2.J1_9 (PA6); no longer U2.J3_10 (PF1)
- net C_BEMF: now also Cb3.1, Cgnd3.1, J_TP5.3 (Pin_3), RdivC1.1, RdivC2.1, U1.8 (3IN-)
- net DUTY: now also U2.J1_2 (PB5), J_TP2.1 (Pin_1); no longer U2.J3_3 (PD0)
- net FASE_A: now also J2.3 (Pin_3), J_TP4.1 (Pin_1), J_TPA1.2 (Pin_2), RdivA2.2, Rstar_A1.1; no longer J2.1 (Pin_1)
- net FASE_B: now also J_TP3.1 (Pin_1), J_TPB1.2 (Pin_2), RdivB2.2, Rstar_B1.1
- net FASE_C: now also J2.1 (Pin_1), J_TP5.2 (Pin_2), J_TPC1.2 (Pin_2), RdivC2.2, Rstar_C1.1; no longer J2.3 (Pin_3)
- net GHA: now also J_TPA1.4 (Pin_4)
- net GHB: now also J_TPB1.4 (Pin_4)
- net GHC: now also J_TPC1.4 (Pin_4)
- net GLA: now also J_TPA1.1 (Pin_1)
- net GLB: now also J_TPB1.1 (Pin_1)
- net GLC: now also J_TPC1.1 (Pin_1)
- net GND: now also CCDES1.2, CDESCOMP1.2, Cgnd1.2, Cgnd2.2, Cgnd3.2, J_TP1.2 (Pin_2), J_TP2.3 (Pin_3), J_TP5.4 (Pin_4), J_TPG1.1 (Pin_1), J_TPG1.2 (Pin_2), J_TPG2.1 (Pin_1), J_TPG2.2 (Pin_2), J_TPG3.1 (Pin_1), J_TPG3.2 (Pin_2), RdivA1.2, RdivB1.2, RdivC1.2, U1.11 (4IN+), U1.12 (GND); no longer CCDES1.1
- net Neu: now also J_TP3.3 (Pin_3), Rstar_A1.2, Rstar_B1.2, Rstar_C1.2
- net Neu_div: now also Cb1.2, Cb2.2, Cb3.2, J_TP5.1 (Pin_1), U1.5 (2IN+), U1.7 (1IN+), U1.9 (3IN+)
- net SensorA: now also U1.2 (2OUT)
- net SensorB: now also U1.1 (1OUT)
- net SensorC: now also U1.14 (OUT3)
- net VBA: now also J_TPA1.3 (Pin_3)
- net VBB: now also J_TPB1.3 (Pin_3)
- net VBC: now also J_TPC1.3 (Pin_3)
- net VCC: now also CCDES1.1; no longer CCDES1.2
- net RGLB: now reaches MOSFET4.1 (G), RGBL1.1
- net RGHA: now reaches MOSFET1.1 (G), RGAH1.1
- net RGLA: now reaches MOSFET2.1 (G), RGAL1.1
- net Led_node: now reaches LED1.1 (K), R1.1
- net RGHB: now reaches MOSFET3.1 (G), RGBH1.1
- net RGLC: now reaches MOSFET6.1 (G), RGCL1.1
- net RGHC: now reaches MOSFET5.1 (G), RGCH1.1
- net B_Vref: no longer names the net of U2.J3_8 (PE2)
- net C_Vref: no longer names the net of U2.J3_9 (PE3)
- no-connect marks 21 -> 23
Other:
- note added: "Calen resistencies de pull up pel SPI?"
- note added: "SUPORT DE LA PLACA"
- note added: "Segur q son 10uF??? mirar si cal canviar petjada"
- note removed: "1N4149: pics de carrega de Cboot < 1 us (IFSM 4 A @1 us); mitjana ~mA. OK."
- note removed: "NOTES DE DISSENY (valors verificats) VCC = 12 V. Buck AP1509-50 -> +5V; LDO LMS8117-3.3 -> +3V3 (alimenta la LaunchPad pel pin +3.3V). Driver: R_in=33R + 100 pF (tau=3.3 ns); Rg=33R -> t_on~Qg/Io+=325 ns, t_off~186 ns. Cboot=1 uF X7R: dV=(Qg+Iqbs*t)/C = 0.31 V per 2.4 ms (fase OL mes llarga). Cboot ceramic, no electrolitic. Shunt 10 mohm 2512: 0.25 W @5 A. Divisor BEMF 39k/3.3k = 0.078 -> 0.94 V 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"
- note removed: "Nomes es poden resistencies E6"
- note removed: "Opamps: buffers (G=1.1) que aillen els divisors d alta impedancia dels comparadors i del filtre."
- note removed: "U2C/U2D no usats: seguidors amb IN+ a GND"
- note removed: "preguntar quina petjada tantal, lm324, capacitat gran"
- company: (none) -> UB
- title: (none) -> Controlador BLDC
- moved on the sheet: CCDES1, RGAH1

Commit message: Versió definitiva de la placa
S'ha fet una revisió de la placa i s'ha canviatt models i disseny en general. És la placa que s'ha enviat a fabricar
Parts:
- removed H4: MountingHole, MountingHole:MountingHole_4.3mm_M4_ISO14580, symbol Mechanical:MountingHole
- removed J_TPG1, J_TPG2, J_TPG3: Conn_01x02_Pin, Connector_PinHeader_2.54mm:PinHeader_1x02_P2.54mm_Vertical, symbol Connector:Conn_01x02_Pin
- removed L1: CDRH127_LDNP-470MC, CDRH127-LDNP-470MC:INDPM120120X800N, symbol CDRH127-LDNP-470MC:CDRH127_LDNP-470MC
- removed U1: LM339DR, LM339DR:D14, symbol LM339DR:LM339DR
- removed U3, U4, U5: IR2301SPBF, IR2301SPBF:SOIC8L_INF, symbol IR2301SPBF:IR2301SPBF
- added IC3: LM339D, LM339D:SOIC127P600X175-14N, symbol LM339D:LM339D
- added IC4, IC5, IC6: IR2301SPBF, IR2301SPBF_modifed:SOIC127P600X175-8N, symbol IR2301SPBF_modifed:IR2301SPBF
- added J3: Conn_01x01_Pin, Connector_PinHeader_2.54mm:PinHeader_1x01_P2.54mm_Vertical, symbol Connector:Conn_01x01_Pin
- added J_TP6: Conn_01x02_Pin, Connector_PinHeader_2.54mm:PinHeader_1x02_P2.54mm_Vertical, symbol Connector:Conn_01x02_Pin
- added J_TPG1, J_TPG2, J_TPG3: Conn_01x04_Pin, Connector_PinHeader_2.54mm:PinHeader_1x04_P2.54mm_Vertical, symbol Connector:Conn_01x04_Pin
- added L1: 744770147, 744770147:WE-PD_1260_1245_1280_121054, symbol 744770147:744770147
- H1, H2, H3: footprint MountingHole:MountingHole_4.3mm_M4_ISO14580 -> MountingHole:MountingHole_3.2mm_M3
- J_DC1: footprint TerminalBlock:TerminalBlock_bornier-2_P5.08mm -> TerminalBlock_Phoenix_MKDS-1,5-2-5.08_1x02_P5.08mm_Horizontal
- RPOT1: footprint TerminalBlock:TerminalBlock_bornier-3_P5.08mm -> TerminalBlock_Phoenix:TerminalBlock_Phoenix_MKDS-1,5-3-5.08_1x03_P5.08mm_Horizontal
- renumbered D4 to D2, D2 to D3, D3 to D4, J_TP5 to J_TP3, J_TP3 to J_TP5, U2 to U1
Connections:
- net +3V3: now also J3.1 (Pin_1)
- net +5V: now also IC3.10 (4IN-), IC3.3 (VCC), L1.1
- net A_BEMF: now also IC3.4 (2IN-)
- net BUCKO: now also L1.2
- net B_BEMF: now also IC3.6 (1IN-)
- net C_BEMF: now also IC3.8 (3IN-)
- net FASE_A: now also IC6.6 (VS)
- net FASE_B: now also IC4.6 (VS)
- net FASE_C: now also IC5.6 (VS)
- net GHA: now also IC6.7 (HO)
- net GHB: now also IC4.7 (HO)
- net GHC: now also IC5.7 (HO)
- net GLA: now also IC6.5 (LO)
- net GLB: now also IC4.5 (LO)
- net GLC: now also IC5.5 (LO)
- net GND: now also IC3.11 (4IN+), IC3.12 (GND), IC4.4 (COM), IC5.4 (COM), IC6.4 (COM), J_TP6.2 (Pin_2), J_TPG1.1 (Pin_1), J_TPG1.4 (Pin_4), J_TPG2.1 (Pin_1), J_TPG2.4 (Pin_4), J_TPG3.1 (Pin_1), J_TPG3.4 (Pin_4)
- net HinA: now also IC6.2 (HIN)
- net HinB: now also IC4.2 (HIN)
- net HinC: now also IC5.2 (HIN)
- net LinA: now also IC6.3 (LIN)
- net LinB: now also IC4.3 (LIN)
- net LinC: now also IC5.3 (LIN)
- net Neu_div: now also IC3.5 (2IN+), IC3.7 (1IN+), IC3.9 (3IN+)
- net SPI_CS: now also U1.J2_9 (PA3); no longer U1.J1_8 (PA5)
- net SPI_MOSI: now also U1.J1_8 (PA5); no longer U1.J2_9 (PA3)
- net SensorA: now also U1.J3_6 (PD3), IC3.2 (2OUT); no longer U1.J3_4 (PD1)
- net SensorB: now also IC3.1 (1OUT)
- net SensorC: now also U1.J3_4 (PD1), IC3.14 (OUT3); no longer U1.J3_6 (PD3)
- net VBA: now also IC6.8 (VB)
- net VBB: now also IC4.8 (VB)
- net VBC: now also IC5.8 (VB)
- net VCC: now also IC4.1 (VCC), IC5.1 (VCC), IC6.1 (VCC), J_TP6.1 (Pin_1)
- net RGHA renamed MGHA
- net MGHA: now also J_TPG3.2 (Pin_2)
- net RGHB renamed MGHB
- net MGHB: now also J_TPG2.2 (Pin_2)
- net RGHC renamed MGHC
- net MGHC: now also J_TPG1.2 (Pin_2)
- net RGLA renamed MGLA
- net MGLA: now also J_TPG3.3 (Pin_3)
- net RGLB renamed MGLB
- net MGLB: now also J_TPG2.3 (Pin_3)
- net RGLC renamed MGLC
- net MGLC: now also J_TPG1.3 (Pin_3)
Other:
- note removed: "Diode Vout->Vin LDO: no cal (Cout=10 uF << 1000 uF, datasheet LMS8117A)."
- note removed: "Segur q son 10uF??? mirar si cal canviar petjada"
- moved on the sheet: CBUCKDESO1, D2, D3, D4, RPull3

Commit message: Reordenat de blocs
Other:
- note removed: "Calen resistencies de pull up pel SPI?"
- note removed: "Condensadors de tantal (petjada temporal)"
- moved on the sheet: CADES1, CADES2, CAH1, CAL1, CA_BOOT1, CBD1, CBD2, CBDES1, CBDES2, CBH1, CBL1, CBUCKDESO1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
